Commit message: Adjust gripper rotation

File: RL-Maniskill/kinova_gen3/Gen3-with-gripper.urdf (robot description, URDF)
Before this commit: robot robotiq_arg2f_85_model, 23 links, 22 joints
Joints:
- joint stack_joint: origin xyz=0 0 -0.06 rpy=3.14159265359 0 0 -> xyz=0 0 -0.06 rpy=3.14159265359 0 1.57079633

Commit message: Update maniskill env

File: RL-Maniskill/kinova_gen3/Gen3-with-gripper.urdf (robot description, URDF)
Before this commit: robot robotiq_arg2f_85_model, 23 links, 22 joints
Joints:
- joint end_effector: origin xyz=0 0 -0.0615250000000001 rpy=3.14159265358979 1.09937075168372E-32 0 -> xyz=0 0 -0.22 rpy=3.14159265358979 1.09937075168372E-32 0
